File: LPSN_LowPowerSensorNode/LPSN/LPSN.kicad_sch (KiCad schematic)
At the start: 8 parts, among them U2 SHT4x, U3 LPS22HB, U5 STM32U031F6Px, Y1 LSC

Commit message: LPSN - backup backup
Parts:
- U4: value ~ -> (none)
